File: KiCAD_files/microcontroller_mini.kicad_sch (KiCad schematic)
At the start: 37 parts, among them J1 Conn_02x20_Top_Bottom, J101 Conn_01x05_Male, J102 Conn_01x06_Male, J2 USB_C_Receptacle_USB2.0, J8 FTSH-107-01-F-DV-K, SW1 KMR241NGLFS, SW2 KMR241NGLFS, U1 STM32G474RE, U3 WE-TVS-82400102, U4 AZ1117-33, Y1 ECS-240-8-37-CKM-TR3 - 24MHz

Commit message: WIP : Implemented fixes to issues from V0.9.
Signed-off-by: Jean Alinei <jean.alinei@laas.fr>
Parts:
- added J103: Conn_01x01, footprints:PinHeader_1x01_P2.54mm_Vertical, symbol Connector_Generic:Conn_01x01
- added R101, R102: 5.1k, Resistor_SMD:R_0402_1005Metric, symbol Device:R_Small
- added T101, T102, T103, T104: Tab, kikit:Tab, symbol PCM_kikit:Tab
- J1: footprint Footprints:RasberryPi Pico -> Footprints:RasberryPi Pico_test
- JP1: footprint Jumper:SolderJumper-2_P1.3mm_Open_TrianglePad1.0x1.5mm -> Resistor_SMD:R_0402_1005Metric
- SW1, SW2: value KMR241NGLFS -> PTS815 SJM 250 SMTR LFS; footprint Button_Switch_SMD:SW_Push_1P1T_NO_CK_KMR2 -> Footprints:SW_SPST_PTS810; Manf# KMR241NGLFS -> PTS815 SJM 250 SMTR LFS
Connections:
- net GNDD: now also R101.1, R102.1
- net NRST: now also J103.1 (Pin_1)
- net at J2.A5 (CC1): now also R102.2
- net at J2.B5 (CC2): now also R101.2
- no-connect marks 9 -> 7
Other:
- note added: "USB C configuration channels resistors"
- title: MCU Shield Board Scheme V1.1.2 -> SPIN V0.9

Commit message: silkscreen fine tuning.
Signed-off-by: Jean Alinei <jean.alinei@laas.fr>
Other:
- company: https://gitlab.laas.fr/owntech/1leg/-/tree/V1.1.2/KiCAD_files -> https://gitlab.laas.fr/owntech/boards/SPIN
- title: SPIN V0.9 -> SPIN V1.0.0
Changed lines of the file:
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@@
   (paper "A3")
   (title_block
-    (title "SPIN V0.9")
+    (title "SPIN V1.0.0")
     (date "2021-06-04")
-    (company "https://gitlab.laas.fr/owntech/1leg/-/tree/V1.1.2/KiCAD_files")
+    (company "https://gitlab.laas.fr/owntech/boards/SPIN")
     (comment 1 "Alinei")
     (comment 2 "Villa")
