File: KiCAD_files/spin.kicad_sch (KiCad schematic)
At the start: 44 parts, among them J1 OwnTech_SPIN, J5 FTSH-107-01-F-DV-K, J6 USB_C_Receptacle_USB2.0, SW1 Push Button, SW2 Push Button, T1 Tab, T2 Tab, T3 Tab, T4 Tab, U1 STM32G474RE, U2 AZ1117-33, U3 WE-TVS-82400102, Y1 ECS-240-8-37-CKM-TR3 - 24MHz

Commit message: changed the 330ohms resistors for the LEDs to 1k
Parts:
- R3, R4: value 330 -> 1k; Manf# CRCW0402330RFKEDC -> RC0402FR-131KL
- TP1, TP2, TP3: now left out of the parts list
Changed lines of the file:
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@@
       (effects (font (size 1.27 1.27)) (justify left))
     )
-    (property "Value" "330" (at 266.065 155.575 0)
+    (property "Value" "1k" (at 266.065 155.575 0)
       (effects (font (size 1.27 1.27)) (justify left))
     )
@@
       (effects (font (size 1.27 1.27)) hide)
     )
-    (property "Datasheet" "https://www.vishay.com/doc?28773" (at 262.89 154.94 0)
-      (effects (font (size 1.27 1.27)) hide)
-    )
-    (property "Manf#" "CRCW0402330RFKEDC" (at 262.89 154.94 0)
+    (property "Datasheet" "https://www.mouser.fr/datasheet/2/447/YAGEO_PYu_RC_Group_51_RoHS_L_12-3313492.pdf" (at 262.89 154.94 0)
+      (effects (font (size 1.27 1.27)) hide)
+    )
+    (property "Manf#" "RC0402FR-131KL" (at 262.89 154.94 0)
       (effects (font (size 1.27 1.27)) hide)
     )
@@
       (effects (font (size 1.27 1.27)) (justify left))
     )
-    (property "Value" "330" (at 247.015 156.21 0)
+    (property "Value" "1k" (at 247.015 156.21 0)
       (effects (font (size 1.27 1.27)) (justify left))
     )
@@
       (effects (font (size 1.27 1.27)) hide)
     )
-    (property "Datasheet" "https://www.vishay.com/doc?28773" (at 243.84 154.94 0)
-      (effects (font (size 1.27 1.27)) hide)
-    )
-    (property "Manf#" "CRCW0402330RFKEDC" (at 243.84 154.94 0)
+    (property "Datasheet" "https://www.mouser.fr/datasheet/2/447/YAGEO_PYu_RC_Group_51_RoHS_L_12-3313492.pdf" (at 243.84 154.94 0)
+      (effects (font (size 1.27 1.27)) hide)
+    )
+    (property "Manf#" "RC0402FR-131KL" (at 243.84 154.94 0)
       (effects (font (size 1.27 1.27)) hide)
     )
@@
   )
   (symbol (lib_id "Connector:TestPoint") (at 387.35 71.12 0) (unit 1)
-    (in_bom yes) (on_board yes) (dnp no) (fields_autoplaced)
+    (in_bom no) (on_board yes) (dnp no) (fields_autoplaced)
     (property "Reference" "TP1" (at 389.89 66.548 0)
       (effects (font (size 1.27 1.27)) (justify left))
@@
       (effects (font (size 1.27 1.27)) hide)
     )
-    (property "Datasheet" "https://www.mouser.fr/datasheet/2/447/PYu_RC_Group_51_RoHS_L_11-1984063.pdf" (at 358.14 53.34 0)
+    (property "Datasheet" "https://www.mouser.fr/datasheet/2/447/YAGEO_PYu_RC_Group_51_RoHS_L_12-3313492.pdf" (at 358.14 53.34 0)
       (effects (font (size 1.27 1.27)) hide)
     )
@@
       (effects (font (size 1.27 1.27)) hide)
     )
-    (property "Datasheet" "https://www.mouser.fr/datasheet/2/447/PYu_RC_Group_51_RoHS_L_11-1984063.pdf" (at 349.25 53.34 0)
+    (property "Datasheet" "https://www.mouser.fr/datasheet/2/447/YAGEO_PYu_RC_Group_51_RoHS_L_12-3313492.pdf" (at 349.25 53.34 0)
       (effects (font (size 1.27 1.27)) hide)
     )
@@
   )
   (symbol (lib_id "Connector:TestPoint") (at 387.35 78.74 180) (unit 1)
-    (in_bom yes) (on_board yes) (dnp no) (fields_autoplaced)
+    (in_bom no) (on_board yes) (dnp no) (fields_autoplaced)
     (property "Reference" "TP3" (at 389.89 80.772 0)
       (effects (font (size 1.27 1.27)) (justify right))
@@
   )
   (symbol (lib_id "Connector:TestPoint") (at 396.24 71.12 0) (unit 1)
-    (in_bom yes) (on_board yes) (dnp no) (fields_autoplaced)
+    (in_bom no) (on_board yes) (dnp no) (fields_autoplaced)
     (property "Reference" "TP2" (at 398.78 66.548 0)
       (effects (font (size 1.27 1.27)) (justify left))

Commit message: Initial commit SPIN V1.2.0
Signed-off-by: Jean Alinei <jean.alinei@laas.fr>
Parts:
- added C15, C16: 10nF, Capacitor_SMD:C_0402_1005Metric, symbol Device:C_Small
- added R8, R9: 100k, Resistor_SMD:R_0402_1005Metric, symbol Device:R
- renumbered D to D1
Connections:
- net GNDD: now also C15.2, C16.2, R8.1, R9.1
- net PB8 renamed PB8-BOOT0
- net PB8-BOOT0: now also C15.1, R8.2
- net PC14 renamed PC14-BOOT1
- net PC14-BOOT1: now also C16.1, R9.2
Other:
- note added: "Capacitor allows to enter bootloader by charging capacitor with PB8-BOOT0 then triggering a software restart."
- note added: "PB8-BOOT0 is non remappable vendor bootloader pin."
- note added: "Pull down resistor prevents entering Bootloader during power up sequence"
- note removed: "I1 is tied to PC1 which is ADC2 CH2 or COMP1 INP (in current mode)"
- note removed: "I2 is tied to PC1 which is ADC1 CH7 or COMP3 INP (in current mode)"
- title: SPIN V1.0.0 -> SPIN V1.2.0

Commit message: SPIN V1.2
Signed-off-by: Jean Alinei <jean.alinei@owntech.org>
Parts:
- removed D1: D_Small_Filled, Diode_SMD:D_SOD-523, symbol Device:D_Small_Filled
- added D1: RB521S30T1G, Diode_SMD:D_SOD-523, symbol Device:D_Schottky
- C1, C2: LCSC C1547 -> (none); Reserved1 (none) -> ea1971f5bd47344ab5e40edded0379fbeeb4e0f8e92933
- C10: LCSC C15195 -> (none); Reserved1 (none) -> 0187ae70d14340d86f04d974ec4c27a5b008d75d8106
- C11, C9: LCSC C15849 -> (none); Reserved1 (none) -> 645fbe0fb770d2555fb2ef4d57fc3d32b98a44297932
- C12, C3, C5, C6, C7, C8: LCSC C1525 -> (none); Reserved1 (none) -> 7b3cb94cdf07e390cf366c3cc999112669ae48b793b17b
- C13, C14: LCSC C15850 -> (none); Reserved1 (none) -> a72de955405c38380bf3e3ac83c8389b843a9beb2e48
- C15, C16: LCSC C1525 -> (none); Manf# VJ0402Y104KXXCW1BC -> CL05B103KB5NNNC; Reserved1 (none) -> 0187ae70d14340d86f04d974ec4c27a5b008d75d8106
- C4: LCSC C19666 -> (none); Reserved1 (none) -> 3d8a9489263d104085f579b50e3ca4d2b659e95e1bed
- F1: value 350mA -> 200mA; Manf# 0ZCK0035FF2G -> 0ZCK0020FF2G; Reserved1 (none) -> 6cbd50413119dedd210b1b5109e0736fee39d08aff48154d
- F2: Reserved1 (none) -> d2c3e8591f8ba933d370fd8bf11e0eb3159fe94b109c4e14
- FB1: Reserved1 (none) -> fa9dc6132c52be12867bf8781b9c760772f915db328b94
- J1, JP1, T1, T2, T3, T4, TP1, TP2, TP3: now not fitted
- J5: Reserved1 (none) -> 6a4bd15f720b85e8304b0d23a2845cf9bf9bbcb9b1fb8d98
- J6: LCSC C165948 -> (none); Reserved1 (none) -> 0e39fec2e5502568bf6ec46f11efde074c48603fbf1964
- LED1, LED2: LCSC C84256 -> (none); Reserved1 (none) -> b7c8193fc17838da8f8700e79654c1ad9c256f308ed662e0
- R1: LCSC C25091 -> (none); Reserved1 (none) -> 94b17578c4c0375b4f05339ee20d2d0d6725e6e349b5
- R2, R7: LCSC C25076 -> (none); Reserved1 (none) -> f7bda095c7a22f5a7b9fb267f63bc7db6f30307ee0a7
- R3, R4: LCSC C25104 -> (none); Reserved1 (none) -> 9fe540edcf7ebac1872c35b3dcde2846ce7b7135a530
- R5, R6: Reserved1 (none) -> 33076a3a1099e7c641a9368fbe7ce1528a418027895d
- R8, R9: LCSC C25091 -> (none); Manf# CR0402-FX-2200GLF -> 0402WGF1003TCE; Reserved1 (none) -> ba0f2a376e26f30a6ac1d204b86f6a0c21139e61d9c1
- SW1, SW2: Reserved1 (none) -> 7aeae425a5712834e40376b9ec7a05ebec6147b6ef1fbb18
- U1: Reserved1 (none) -> 70742f000f1395159f1f637dd92a9ca5bb7bb9665866bf
- U2: LCSC C6186 -> (none); Reserved1 (none) -> e057f1cf1197ccaf308393a6f6a50ccc557d2682b00360
- U3: Reserved1 (none) -> eced9b9d3e64f8dafdb949ec9c5c3a9bc86d14298709e1ad
- Y1: Reserved1 (none) -> 5cd0b49329b07fb352943c2ba2c979a68a3824ce0636a907
Connections:
- net VBUS: now also D1.2 (A)
- net at F2.2: now also D1.1 (K)

Commit message: Minor SPIN revision, bumping to v1.2.1 - Silkscreen improvements.
Signed-off-by: Jean Alinei <jean.alinei@owntech.org>
Parts:
- added G1: LOGO, Footprints:owntech_mini8, symbol Symbols:LOGO
- F2: Reserved1 d2c3e8591f8ba933d370fd8bf11e0eb3159fe94b109c4e14 -> e394ed3fe5d0680e1c8a20637c48b7aa36891a7c49fe93
- FB1: Reserved1 fa9dc6132c52be12867bf8781b9c760772f915db328b94 -> 54a61a2086c15f84846f2b37f37a9f22d66b0f494102
- J5: value FTSH-107-01-F-DV-K -> FTSH-107-01-F-DV-K; Reserved1 6a4bd15f720b85e8304b0d23a2845cf9bf9bbcb9b1fb8d98 -> 2b27be521c8cdac1386794cac7f88b156d1af3996629da40
- R7: Reserved1 f7bda095c7a22f5a7b9fb267f63bc7db6f30307ee0a7 -> 3d1976e3817e90c0187ecb328e058dc5f7fd0066caab
- SW1, SW2: Reserved1 7aeae425a5712834e40376b9ec7a05ebec6147b6ef1fbb18 -> 3d10a0ffc940994c1a0f401a8bb0f8b8d75eee21f7b1ae
- U2: Position Offset (none) -> -0.45,0
- U3: Rotation Offset (none) -> 90
- Y1: Reserved1 5cd0b49329b07fb352943c2ba2c979a68a3824ce0636a907 -> ed5b21bbfd07a4133b307b5a996b2180e979235b0a3bbf6096
Other:
- note added: "Global nets indicate user-accessible signals."
- note removed: "Global net are used to symbolize user accessible signals"
- title: SPIN V1.2.0 -> SPIN V1.2.1
- moved on the sheet: C13, C14, R7, T1, T2, T3, T4
